File: pcb/kagu/kagu.kicad_pcb (KiCad board)
At the start: 2 copper layers, 43 parts, among them J1 Conn_01x04_Pin, SW1 SW_Push, SW10 SW_Push, SW11 SW_Push, SW12 SW_Push, SW13 SW_Push, SW14 SW_Push, SW15 SW_Push, SW16 SW_Push, SW17 SW_Push, SW18 SW_Push, SW2 SW_Push, SW3 SW_Push, SW4 SW_Push, SW5 SW_Push, SW6 SW_Push, SW7 SW_Push, SW8 SW_Push, SW9 SW_Push, U1 XIAO-nRF52840-Plus-SMD

Commit message: feat(pcb): make a first no error version
Parts:
- added R1: R(1k), Resistor_SMD:R_0805_2012Metric, F.Cu at (177.7, 101.5)
- D1: renamed from D15; footprint Diode_SMD:D_SOD-123 -> kagu:D_SOD-123
- D10: renamed from D2; footprint Diode_SMD:D_SOD-123 -> kagu:D_SOD-123
- D11: renamed from D17; footprint Diode_SMD:D_SOD-123 -> kagu:D_SOD-123
- D12: renamed from D13; footprint Diode_SMD:D_SOD-123 -> kagu:D_SOD-123
- D13: renamed from D9; footprint Diode_SMD:D_SOD-123 -> kagu:D_SOD-123
- D14: renamed from D6; footprint Diode_SMD:D_SOD-123 -> kagu:D_SOD-123
- D15: renamed from D3; footprint Diode_SMD:D_SOD-123 -> kagu:D_SOD-123
- D16: renamed from D18; footprint Diode_SMD:D_SOD-123 -> kagu:D_SOD-123
- D17: renamed from D14; footprint Diode_SMD:D_SOD-123 -> kagu:D_SOD-123
- D18: renamed from D10; footprint Diode_SMD:D_SOD-123 -> kagu:D_SOD-123
- D2: renamed from D11; footprint Diode_SMD:D_SOD-123 -> kagu:D_SOD-123
- D3: renamed from D7; footprint Diode_SMD:D_SOD-123 -> kagu:D_SOD-123
- D4, D8: footprint Diode_SMD:D_SOD-123 -> kagu:D_SOD-123
- D5: renamed from D1; footprint Diode_SMD:D_SOD-123 -> kagu:D_SOD-123
- D6: renamed from D16; footprint Diode_SMD:D_SOD-123 -> kagu:D_SOD-123
- D7: renamed from D12; footprint Diode_SMD:D_SOD-123 -> kagu:D_SOD-123
- D9: renamed from D5; footprint Diode_SMD:D_SOD-123 -> kagu:D_SOD-123
- moved D16 166.4 mm to (169.4, 126.1), turned to -30 degrees
- moved D17 159.6 mm to (146.0, 111.9), turned to -110 degrees
- moved D12 147.5 mm to (149.0, 94.0), turned to 90 degrees
- moved D11 147.1 mm to (167.0, 96.0), turned to 90 degrees
- moved D7 139.0 mm to (149.0, 77.0), turned to 90 degrees
- moved D6 137.4 mm to (167.0, 79.0), turned to 90 degrees
- moved D2 131.4 mm to (149.0, 60.0), turned to 90 degrees
- moved D1 128.4 mm to (167.0, 62.0), turned to 90 degrees
- moved Battery_LED1 124.8 mm to (176.5, 106.5), turned to 60 degrees
- moved U1 124.7 mm to (181.7, 64.0), turned to 90 degrees
- moved GND_Pad1 117.4 mm to (173.0, 79.5), turned to -90 degrees
- moved Switch1 115.3 mm to (186.5, 90.5)
- moved Battery1 115.1 mm to (176.5, 90.5)
- moved Battery_Pad1 114.2 mm to (173.0, 77.5), turned to -90 degrees
- moved SW1 84.1 mm to (158.0, 61.0)
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- renumbered SW15 to SW1, SW2 to SW10, SW17 to SW11, SW13 to SW12, SW9 to SW13, SW6 to SW14, SW3 to SW15, SW18 to SW16, SW14 to SW17, SW10 to SW18, SW11 to SW2, SW7 to SW3, SW1 to SW5, SW16 to SW6, SW12 to SW7, SW5 to SW9
Connections:
- U1 pad 28: +BATT -> unconnected-(U1-VBAT-Pad28)
- U1 pad 29: GND -> unconnected-(U1-GND-Pad29)
Routing:
- net row1: track 0.00 -> 139.6 mm, vias 0 -> 9
- net row3: track 0.00 -> 136.3 mm, vias 0 -> 5
- net row2: track 0.00 -> 133.8 mm, vias 0 -> 9
- net col5: track 0.00 -> 131.8 mm, vias 0 -> 1
- net row4: track 0.00 -> 121.5 mm, vias 0 -> 5
- net col3: track 0.00 -> 120.2 mm, vias 0 -> 1
- net col4: track 0.00 -> 110.1 mm, vias 0 -> 1
- net col2: track 0.00 -> 95.3 mm, vias 0 -> 1
- net col1: track 0.00 -> 85.3 mm, vias 0 -> 1
- net GND: track 0.00 -> 71.5 mm, vias 0 -> 2
- net +BATT: track 0.00 -> 37.2 mm
- net Net-(D18-A): track 0.00 -> 18.2 mm
- net Net-(D17-A): track 0.00 -> 16.3 mm
- net Net-(D16-A): track 0.00 -> 16.1 mm
- net Net-(D4-A): track 0.00 -> 14.1 mm
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Other:
- board outline added: 114.5 x 88.9 mm

Commit message: feat(pcb): send to prod for one half (gl)
Parts:
- removed J1: Conn_01x04_Pin, Connector_JST:JST_SH_SM04B-SRSS-TB_1x04-1MP_P1.00mm_Horizontal
- added H1: MountingHole, MountingHole:MountingHole_3.2mm_M3_DIN965_Pad, F.Cu at (194.5, 55.5)
- added H2: MountingHole, MountingHole:MountingHole_3.2mm_M3_DIN965_Pad, F.Cu at (193.0, 99.0)
- added H3: MountingHole, MountingHole:MountingHole_3.2mm_M3_DIN965_Pad, F.Cu at (162.5, 125.0)
- added H4: MountingHole, MountingHole:MountingHole_3.2mm_M3_DIN965_Pad, F.Cu at (116.0, 99.0)
- added H5: MountingHole, MountingHole:MountingHole_3.2mm_M3_DIN965_Pad, F.Cu at (74.5, 109.0)
- added H6: MountingHole, MountingHole:MountingHole_3.2mm_M3_DIN965_Pad, F.Cu at (74.5, 64.5)
- added H7: MountingHole, MountingHole:MountingHole_3.2mm_M3_DIN965_Pad, F.Cu at (165.5, 106.5)
- added I2S_SCK1: Conn_01x01_Pin, kagu:TestPad, F.Cu at (194.5, 91.5)
- added I2S_SD1: Conn_01x01_Pin, kagu:TestPad, F.Cu at (194.5, 94.5)
- added I2S_WS1: Conn_01x01_Pin, kagu:TestPad, F.Cu at (194.5, 88.5)
- added NFC_1: Conn_01x01_Pin, kagu:TestPad, F.Cu at (194.5, 84.5)
- added NFC_2: Conn_01x01_Pin, kagu:TestPad, F.Cu at (194.5, 81.5)
- added RESET_HW1: Conn_01x01_Pin, kagu:TestPad, F.Cu at (173.0, 80.5)
- added SPI_MISO1: Conn_01x01_Pin, kagu:TestPad, F.Cu at (194.5, 68.5)
- added SPI_MOSI1: Conn_01x01_Pin, kagu:TestPad, F.Cu at (194.5, 65.5)
- added SPI_SCK1: Conn_01x01_Pin, kagu:TestPad, F.Cu at (194.5, 71.5)
- added SW19: SW_Push, Button_Switch_SMD:SW_Push_SPST_NO_Alps_SKRK, F.Cu at (187.0, 102.0)
- added UART_RX1: Conn_01x01_Pin, kagu:TestPad, F.Cu at (194.5, 75.0)
- added UART_TX1: Conn_01x01_Pin, kagu:TestPad, F.Cu at (194.5, 78.0)
- Bat_HW1: renamed from Battery_Pad1; footprint Connector_Wire:SolderWirePad_1x01_SMD_1x2mm -> kagu:TestPad
- GND_HW1: renamed from GND_Pad1; footprint Connector_Wire:SolderWirePad_1x01_SMD_1x2mm -> kagu:TestPad
- U1: footprint XIAO nRF52840:XIAO-nRF52840-Plus-SMD -> XIAO nRF52840:XIAO-23P-Add-On-Plus
- moved Bat_HW1 6.52 mm to (179.5, 77.0), turned to 0 degrees
- moved GND_HW1 2.50 mm to (173.0, 77.0), turned to 0 degrees
- renumbered Battery1 to Bat_Con1, Battery_LED1 to Bat_LED_Con1, Switch1 to Switch_Con1
Connections:
- U1 pad 10: row2 -> row3
- U1 pad 11: row1 -> row4
- U1 pad 15: unconnected-(U1-D11-Pad15) -> i2s sd
- U1 pad 16: unconnected-(U1-D12-Pad16) -> i2s sck
- U1 pad 17: unconnected-(U1-D13-Pad17) -> i2s ws
- U1 pad 18: unconnected-(U1-D14-Pad18) -> nfc 1
- U1 pad 19: unconnected-(U1-D15-Pad19) -> nfc 2
- U1 pad 21: unconnected-(U1-D17-Pad21) -> spi sck
- U1 pad 22: unconnected-(U1-D18-Pad22) -> spi miso
- U1 pad 23: unconnected-(U1-D19-Pad23) -> spi mosi
- U1 pad 6: unconnected-(U1-D5-Pad6) -> uart tx
- U1 pad 7: unconnected-(U1-D6-Pad7) -> uart rx
- U1 pad 8: row4 -> row1
- U1 pad 9: row3 -> row2
Routing:
- net GND: track 71.5 -> 2.00 mm, vias 2 -> 1
- net i2s sd: track 0.00 -> 54.5 mm
- net i2s sck: track 0.00 -> 50.3 mm
- net i2s ws: track 0.00 -> 45.5 mm
- net nfc 1: track 0.00 -> 42.6 mm
- net nfc 2: track 0.00 -> 41.4 mm
- net uart tx: track 0.00 -> 31.1 mm
- net reset: track 0.00 -> 30.9 mm, vias 0 -> 1
- net uart rx: track 0.00 -> 26.7 mm
- net row4: track 121.5 -> 134.0 mm, vias 5 -> 4
- net col5: track 131.8 -> 121.3 mm, vias 1 -> 0
- net row3: track 136.3 -> 141.5 mm
- net +BATT: track 37.2 -> 32.1 mm, vias 0 -> 1
- net spi sck: track 0.00 -> 4.41 mm
- net spi miso: track 0.00 -> 4.22 mm
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- added copper zone on F.Cu, net GND
Other:
- board size 114.5 x 88.9 mm -> 127 x 91.5 mm
