File: pcb/kagu/kagu.kicad_sch (KiCad schematic)
At the start: 44 parts, among them J1 Conn_01x04_Pin, SW1 SW_Push, SW10 SW_Push, SW11 SW_Push, SW12 SW_Push, SW13 SW_Push, SW14 SW_Push, SW15 SW_Push, SW16 SW_Push, SW17 SW_Push, SW18 SW_Push, SW2 SW_Push, SW3 SW_Push, SW4 SW_Push, SW5 SW_Push, SW6 SW_Push, SW7 SW_Push, SW8 SW_Push, SW9 SW_Push, U1 XIAO-nRF52840-Plus-SMD

Commit message: feat(pcb): make a first no error version
Parts:
- D1: renamed from D15; footprint Diode_SMD:D_SOD-123 -> kagu:D_SOD-123
- D10: renamed from D2; footprint Diode_SMD:D_SOD-123 -> kagu:D_SOD-123
- D11: renamed from D17; footprint Diode_SMD:D_SOD-123 -> kagu:D_SOD-123
- D12: renamed from D13; footprint Diode_SMD:D_SOD-123 -> kagu:D_SOD-123
- D13: renamed from D9; footprint Diode_SMD:D_SOD-123 -> kagu:D_SOD-123
- D14: renamed from D6; footprint Diode_SMD:D_SOD-123 -> kagu:D_SOD-123
- D15: renamed from D3; footprint Diode_SMD:D_SOD-123 -> kagu:D_SOD-123
- D16: renamed from D18; footprint Diode_SMD:D_SOD-123 -> kagu:D_SOD-123
- D17: renamed from D14; footprint Diode_SMD:D_SOD-123 -> kagu:D_SOD-123
- D18: renamed from D10; footprint Diode_SMD:D_SOD-123 -> kagu:D_SOD-123
- D2: renamed from D11; footprint Diode_SMD:D_SOD-123 -> kagu:D_SOD-123
- D3: renamed from D7; footprint Diode_SMD:D_SOD-123 -> kagu:D_SOD-123
- D4, D8: footprint Diode_SMD:D_SOD-123 -> kagu:D_SOD-123
- D5: renamed from D1; footprint Diode_SMD:D_SOD-123 -> kagu:D_SOD-123
- D6: renamed from D16; footprint Diode_SMD:D_SOD-123 -> kagu:D_SOD-123
- D7: renamed from D12; footprint Diode_SMD:D_SOD-123 -> kagu:D_SOD-123
- D9: renamed from D5; footprint Diode_SMD:D_SOD-123 -> kagu:D_SOD-123
- R1: footprint (none) -> Resistor_SMD:R_0805_2012Metric
- renumbered SW15 to SW1, SW2 to SW10, SW17 to SW11, SW13 to SW12, SW9 to SW13, SW6 to SW14, SW3 to SW15, SW18 to SW16, SW14 to SW17, SW10 to SW18, SW11 to SW2, SW7 to SW3, SW1 to SW5, SW16 to SW6, SW12 to SW7, SW5 to SW9
Connections:
- net +BATT: no longer U1.28 (VBAT)
- net GND: no longer U1.29 (GND)
- no-connect marks 20 -> 22
Other:
- note added: "Hand wired"

Commit message: feat(pcb): send to prod for one half (gl)
Parts:
- removed J1: Conn_01x04_Pin, Connector_JST:JST_SH_SM04B-SRSS-TB_1x04-1MP_P1.00mm_Horizontal, symbol Connector:Conn_01x04_Pin
- added H1, H2, H3, H4, H5, H6, H7: MountingHole, MountingHole:MountingHole_3.2mm_M3_DIN965_Pad, symbol Mechanical:MountingHole
- added I2S_SCK1, I2S_SD1, I2S_WS1, NFC_1, NFC_2, RESET_HW1, SPI_MISO1, SPI_MOSI1, SPI_SCK1, UART_RX1, UART_TX1: Conn_01x01_Pin, kagu:TestPad, symbol Connector:Conn_01x01_Pin
- added SW19: SW_Push, Button_Switch_SMD:SW_Push_SPST_NO_Alps_SKRK, symbol Switch:SW_Push
- Bat_HW1: renamed from Battery_Pad1; footprint Connector_Wire:SolderWirePad_1x01_SMD_1x2mm -> kagu:TestPad
- GND_HW1: renamed from GND_Pad1; footprint Connector_Wire:SolderWirePad_1x01_SMD_1x2mm -> kagu:TestPad
- U1: footprint XIAO nRF52840:XIAO-nRF52840-Plus-SMD -> XIAO nRF52840:XIAO-23P-Add-On-Plus
- renumbered Battery1 to Bat_Con1, Battery_LED1 to Bat_LED_Con1, Switch1 to Switch_Con1
Connections:
- net GND: now also SW19.2
- net row1: now also U1.8 (D7); no longer U1.11 (D10)
- net row2: now also U1.9 (D8); no longer U1.10 (D9)
- net row3: now also U1.10 (D9); no longer U1.9 (D8)
- net row4: now also U1.11 (D10); no longer U1.8 (D7)
- net i2s sd: now reaches U1.15 (D11)
- net i2s sd: now also I2S_SD1.1 (Pin_1)
- net i2s sck: now reaches U1.16 (D12)
- net i2s sck: now also I2S_SCK1.1 (Pin_1)
- net i2s ws: now reaches U1.17 (D13)
- net i2s ws: now also I2S_WS1.1 (Pin_1)
- net nfc 1: now reaches U1.18 (D14)
- net nfc 1: now also NFC_1.1 (Pin_1)
- net nfc 2: now reaches U1.19 (D15)
- net nfc 2: now also NFC_2.1 (Pin_1)
- net spi sck: now reaches U1.21 (D17)
- net spi sck: now also SPI_SCK1.1 (Pin_1)
- net spi miso: now reaches U1.22 (D18)
- net spi miso: now also SPI_MISO1.1 (Pin_1)
- net spi mosi: now reaches U1.23 (D19)
- net spi mosi: now also SPI_MOSI1.1 (Pin_1)
- net uart tx: now reaches U1.6 (D5)
- net uart tx: now also UART_TX1.1 (Pin_1)
- net uart rx: now reaches U1.7 (D6)
- net uart rx: now also UART_RX1.1 (Pin_1)
- new net reset: RESET_HW1.1 (Pin_1), SW19.1
- no-connect marks 22 -> 8
Other:
- note added: "Battery Logic"
- note added: "Controller Placeholder"
- note added: "Key Matrix"
- note added: "Reset Button"
- note added: "Test Pads"
- moved on the sheet: Bat_Con1, Bat_HW1, Bat_LED_Con1, D1, D10, D11, D12, D13, D14, D15, D16, D17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
